File: Hardware/CristmasVillage Driver 1-3.sch (EAGLE design)
At the start: 56 parts, among them CN1 MJ-180SMT, CN2-PROG JST-6PSPI-SIDE-S6B, CN3-SERIAL JST-4PSIDE-S4B, CN5-LEDSTRIPS HDR_2X10_SIDE-MOUNT, IC1 UA78M05DCY, IC2 LM358D, IC3 LM358D, IC4 LM358D, IC5 ATTINY-4/5/9/10, IC6 TINY2313-*S*, Q1 Si2309CD, Q10 NX7002AKW, Q11 NX7002AKW, Q12 NX7002AKW, Q2 NX7002AKW, Q3 NX7002AKW, Q4 NX7002AKW, Q5 NX7002AKW, Q6 NX7002AKW, Q7 NX7002AKW, Q8 NX7002AKW, Q9 NX7002AKW, SW1 POWER, SW2 NIGHT-MODE

Commit message: Cleaned up silkscreen - added gerber exports
Connections:
- net N$4 renamed RX
- net N$5 renamed TX
Changed lines of the file:
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@@
 </segment>
 </net>
-<net name="N$4" class="0">
+<net name="RX" class="0">
 <segment>
 <pinref part="CN3-SERIAL" gate="G$1" pin="2"/>
@@
 </segment>
 </net>
-<net name="N$5" class="0">
+<net name="TX" class="0">
 <segment>
 <pinref part="CN3-SERIAL" gate="G$1" pin="3"/>
